File: hardware/bicicletta-power.brd (EAGLE design)
At the start: 160 x 100 mm, 23 parts, among them IC1 LM5017, IC2 LM1117-3.3

Commit message: First final draft of PCB layout. Requires validation.
Parts:
- moved IC2 6.38 mm to (82.5, 74.3)
- moved C1 6.38 mm to (81.3, 67.3)
- moved C2 6.38 mm to (81.3, 81.3)
Routing:
- net 3.3V: track 0.00 -> 14.3 mm
- net 5V: track 7.78 -> 19.0 mm
- net GND: track 7.55 -> 12.2 mm
Changed lines of the file:
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@@
 <element name="L1" library="rcl" package="L1812" value="100uH" x="68.58" y="73.66" rot="MR180"/>
 <element name="R_R" library="rcl" package="M0805" value="2M" x="64.77" y="75.565"/>
-<element name="IC2" library="SparkFun-PowerIC" package="SOT223" value="LM1117-3.3" x="88.9" y="73.66" rot="R270"/>
-<element name="C1" library="rcl" package="UD-5X5,8_NICHICON" value="14uF" x="87.63" y="66.675" rot="R180"/>
-<element name="C2" library="rcl" package="UD-5X5,8_NICHICON" value="14uF" x="87.63" y="80.645"/>
+<element name="IC2" library="SparkFun-PowerIC" package="SOT223" value="LM1117-3.3" x="82.55" y="74.295" rot="R270"/>
+<element name="C1" library="rcl" package="UD-5X5,8_NICHICON" value="14uF" x="81.28" y="67.31" rot="R180"/>
+<element name="C2" library="rcl" package="UD-5X5,8_NICHICON" value="14uF" x="81.28" y="81.28"/>
 <element name="C_R" library="rcl" package="C0603" value="3300pF" x="72.0725" y="74.295" rot="R270"/>
 <element name="C_AC" library="rcl" package="C0603" value="100nF" x="68.58" y="74.295" rot="R180"/>
@@
 <polygon width="0.4064" layer="1" thermals="no" rank="2">
 <vertex x="52.07" y="83.82"/>
-<vertex x="77.47" y="83.82"/>
-<vertex x="77.47" y="64.77"/>
+<vertex x="87.63" y="83.82"/>
+<vertex x="87.63" y="64.77"/>
 <vertex x="42.2275" y="64.77"/>
 <vertex x="42.2275" y="70.485"/>
@@
 <wire x1="45.085" y1="79.375" x2="45.085" y2="78.6525" width="1.016" layer="1"/>
 <wire x1="45.085" y1="78.6525" x2="46.0375" y2="77.7" width="1.016" layer="1"/>
-<wire x1="85.8012" y1="75.9714" x2="85.93" y2="80.645" width="0" layer="19" extent="1-1"/>
-<wire x1="76.2" y1="81.915" x2="85.93" y2="80.645" width="0" layer="19" extent="1-1"/>
-<wire x1="89.33" y1="66.675" x2="85.8012" y2="75.9714" width="0" layer="19" extent="1-1"/>
+<wire x1="79.4512" y1="76.6064" x2="79.4512" y2="80.5162" width="0.8128" layer="1"/>
+<wire x1="79.4512" y1="80.5162" x2="79.58" y2="81.28" width="0.8128" layer="1"/>
 </signal>
 <signal name="V_BATT">
@@
 <contactref element="C_OUT" pad="1"/>
 <polygon width="0.4064" layer="1">
-<vertex x="68.58" y="77.47"/>
-<vertex x="76.5175" y="77.47"/>
-<vertex x="76.5175" y="71.4375"/>
+<vertex x="69.215" y="75.2475"/>
+<vertex x="74.93" y="75.2475"/>
+<vertex x="74.93" y="71.4375"/>
 <vertex x="72.7075" y="71.4375"/>
 <vertex x="72.7075" y="70.1675"/>
-<vertex x="68.58" y="70.1675"/>
+<vertex x="69.215" y="70.1675"/>
 </polygon>
 <contactref element="L1" pad="2"/>
@@
 <wire x1="69.85" y1="68.58" x2="69.85" y2="70.8" width="1.016" layer="1"/>
 <wire x1="69.85" y1="70.8" x2="69.8475" y2="70.8025" width="1.016" layer="1"/>
-<wire x1="85.905" y1="66.675" x2="85.8012" y2="71.3486" width="0" layer="19" extent="1-1"/>
-<wire x1="73.66" y1="73.66" x2="85.8012" y2="71.3486" width="0" layer="19" extent="1-1"/>
+<wire x1="73.66" y1="73.66" x2="76.2" y2="73.66" width="0.8128" layer="1"/>
+<wire x1="76.2" y1="73.66" x2="77.8764" y2="71.9836" width="0.8128" layer="1"/>
+<wire x1="79.4512" y1="71.9836" x2="77.8764" y2="71.9836" width="0.8128" layer="1"/>
+<wire x1="79.555" y1="67.31" x2="79.555" y2="71.2448" width="0.8128" layer="1"/>
+<wire x1="79.555" y1="71.2448" x2="79.4512" y2="71.9836" width="0.8128" layer="1"/>
 </signal>
 <signal name="N$1">
@@
 <contactref element="IC2" pad="2"/>
 <contactref element="C2" pad="+"/>
-<wire x1="91.999" y1="73.66" x2="89.355" y2="80.645" width="0" layer="19" extent="1-1"/>
-<wire x1="85.8012" y1="73.66" x2="91.999" y2="73.66" width="0" layer="19" extent="1-1"/>
+<wire x1="85.649" y1="74.295" x2="79.4512" y2="74.295" width="0.8128" layer="1"/>
+<wire x1="85.649" y1="74.295" x2="85.649" y2="78.636" width="0.8128" layer="1"/>
+<wire x1="85.649" y1="78.636" x2="83.005" y2="81.28" width="0.8128" layer="1"/>
 </signal>
 <signal name="N$4">

Commit message: Inductor speced out. PCB placement getting closer.
Parts:
- L1: device rcl:L1812 -> Railstars:SRN1060
- moved L1 11.8 mm to (80.3, 74.3), flipped to the top, turned to 0 degrees
- moved IC2 8.26 mm to (90.8, 74.6)
- moved C1 1.91 mm to (81.3, 65.4), turned to 0 degrees
- moved C2 1.91 mm to (81.3, 83.2)
- moved R_R 1.35 mm to (63.8, 74.6)
- moved R_FB2 1.00 mm to (68.6, 71.8)
- moved R_FB1 0.95 mm to (63.8, 71.8)
- moved C_OUT 0.71 mm to (71.8, 70.8)
- moved C_R 0.45 mm to (71.8, 74.6)
- moved C_AC 0.32 mm to (68.6, 74.6)
- moved C_BST 0.32 mm to (59.4, 74.6)
Connections:
- net 5V: now also L1.P$2; no longer L1.2
- net N$4: now also L1.P$1; no longer L1.1
Routing:
- net N$4: track 17.0 -> 32.6 mm, vias 1 -> 2
- net 3.3V: track 14.3 -> 20.5 mm
- net 5V: track 19.0 -> 24.7 mm, vias 1 -> 0
- net GND: track 12.2 -> 7.55 mm
- net N$2: track 18.9 -> 20.5 mm
Other:
- outline, holes or cut-outs redrawn

Commit message: SMall tweaks that add up.
Parts:
- moved JP4 2.54 mm to (73.0, 78.1)
- moved JP5 2.54 mm to (70.5, 78.1)
Routing:
- net 5V: track 24.7 -> 33.4 mm, vias 0 -> 1
- net SHUNT-: track 15.5 -> 11.7 mm
- net N$2: track 20.5 -> 17.5 mm
- net SHUNT+: track 10.4 -> 11.7 mm
- net N$6: track 8.18 -> 8.96 mm
- net N$4: track 32.6 -> 32.0 mm
- net N$1: track 4.39 -> 4.95 mm
