File: hardware/bicicletta-sensor.brd (EAGLE design)
At the start: 45.7 x 19.1 mm, 3 parts

Commit message: Better analog design. Still working on DAC for throttle output.
Parts:
- added IC1: LMV324MZ, linear:TSSOP14
- added JP1: (no value), SparkFun-Connectors:1X03
- added R1: 60K, rcl:R0603
- added R10, R9: 600, rcl:R0603
- added R2: 3K, rcl:R0603
- added R3: 50K, rcl:R0603
- added R4, R5: 10K, rcl:R0603
- added R6: 5.8K, rcl:R0603
- added R7: 1K, rcl:R0603
- added R8: 2K, rcl:R0603
Connections:
- removed net A0: U$1.P$23
- removed net A1: U$1.P$22
- new net BATTERY_3.3: IC1.1, R3.1, U$1.P$23
- new net BIAS: R4.2, R5.1, R6.2
- new net N$1: IC1.9, R10.2, R9.1
- new net N$11: IC1.6, R7.1, R8.2
- new net N$2: IC1.3, R1.2, R2.1
- new net N$3: IC1.2, R3.2, R4.1
- new net THROTTLE_IN_3.3: IC1.5, IC1.7, U$1.P$22
- new net THROTTLE_IN_5: JP1.2, R7.2
- new net THROTTLE_OUT_3.3: IC1.10, IC1.8, R9.2
- net 3.3V: now also R5.2
- net 5V: now also IC1.4, JP1.3
- net GND: now also IC1.11, JP1.1, R10.1, R2.2, R6.1, R8.1
- net V_BATT: now also R1.1
Routing:
- net V_BATT: track 0.00 -> 18.0 mm
- net 3.3V: track 0.00 -> 17.1 mm
- net BATTERY_3.3: track 0.00 -> 14.7 mm, vias 0 -> 1
- net N$11: track 0.00 -> 6.64 mm
- net N$2: track 0.00 -> 4.86 mm
- net BIAS: track 0.00 -> 2.54 mm
- added copper zone on layer 1, net GND
Changed lines of the file:
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@@
 </element>
 <element name="U$2" library="Artificial Science" package="RAILSTARS_25MM" value="" x="44.45" y="5.08" rot="MR0"/>
+<element name="R1" library="rcl" package="R0603" value="60K" x="15.24" y="6.35" rot="R90"/>
+<element name="R2" library="rcl" package="R0603" value="3K" x="17.78" y="6.35" rot="R270"/>
+<element name="R5" library="rcl" package="R0603" value="10K" x="30.48" y="12.7" rot="R270"/>
+<element name="R6" library="rcl" package="R0603" value="5.8K" x="33.02" y="12.7" rot="R90"/>
+<element name="R7" library="rcl" package="R0603" value="1K" x="30.48" y="6.35" rot="R90"/>
+<element name="R8" library="rcl" package="R0603" value="2K" x="33.02" y="6.35" rot="R270"/>
+<element name="JP1" library="SparkFun-Connectors" package="1X03" value="" x="2.54" y="-5.08"/>
+<element name="IC1" library="linear" package="TSSOP14" value="LMV324MZ" x="-1.27" y="-11.43"/>
+<element name="R9" library="rcl" package="R0603" value="600" x="-3.81" y="-17.78"/>
+<element name="R10" library="rcl" package="R0603" value="600" x="-3.81" y="-22.86"/>
+<element name="R3" library="rcl" package="R0603" value="50K" x="-3.81" y="-27.94"/>
+<element name="R4" library="rcl" package="R0603" value="10K" x="-3.81" y="-33.02"/>
 </elements>
 <signals>
@@
 <vertex x="0" y="0"/>
 </polygon>
+<contactref element="R2" pad="2"/>
+<contactref element="R6" pad="1"/>
+<contactref element="R8" pad="1"/>
+<polygon width="0.4064" layer="1">
+<vertex x="9.525" y="19.05"/>
+<vertex x="45.72" y="19.05"/>
+<vertex x="46.99" y="0"/>
+<vertex x="0" y="0"/>
+<vertex x="0" y="13.97"/>
+<vertex x="5.08" y="13.97"/>
+<vertex x="5.715" y="13.0175"/>
+<vertex x="5.715" y="9.525"/>
+<vertex x="11.43" y="3.81"/>
+<vertex x="16.51" y="3.81"/>
+<vertex x="16.51" y="7.3025"/>
+<vertex x="12.7" y="7.3025"/>
+<vertex x="9.525" y="10.4775"/>
+</polygon>
+<contactref element="JP1" pad="1"/>
+<contactref element="IC1" pad="11"/>
+<contactref element="R10" pad="1"/>
+<wire x1="33.02" y1="11.85" x2="43.18" y2="17.145" width="0" layer="19" extent="1-1"/>
+<wire x1="33.02" y1="7.2" x2="33.02" y2="11.85" width="0" layer="19" extent="1-1"/>
+<wire x1="40.64" y1="1.905" x2="33.02" y2="7.2" width="0" layer="19" extent="1-1"/>
+<wire x1="43.18" y1="1.905" x2="40.64" y2="1.905" width="0" layer="19" extent="1-1"/>
+<wire x1="17.78" y1="5.5" x2="33.02" y2="7.2" width="0" layer="19" extent="1-1"/>
+<wire x1="3.81" y1="13.335" x2="17.78" y2="5.5" width="0" layer="19" extent="1-1"/>
+<wire x1="2.54" y1="-5.08" x2="3.81" y2="13.335" width="0" layer="19" extent="1-1"/>
+<wire x1="-1.27" y1="-8.7122" x2="2.54" y2="-5.08" width="0" layer="19" extent="1-1"/>
+<wire x1="-4.66" y1="-22.86" x2="-1.27" y2="-8.7122" width="0" layer="19" extent="1-1"/>
 </signal>
 <signal name="V_BATT">
 <contactref element="JP3" pad="1"/>
+<contactref element="R1" pad="1"/>
+<wire x1="3.81" y1="15.875" x2="5.715" y2="15.875" width="1.016" layer="1"/>
+<wire x1="5.715" y1="15.875" x2="7.62" y2="13.97" width="1.016" layer="1"/>
+<wire x1="7.62" y1="13.97" x2="7.62" y2="10.16" width="1.016" layer="1"/>
+<wire x1="7.62" y1="10.16" x2="12.38" y2="5.4" width="1.016" layer="1"/>
+<wire x1="15.24" y1="5.5" x2="12.38" y2="5.4" width="1.016" layer="1"/>
 </signal>
 <signal name="5V">
 <contactref element="U$1" pad="P$12"/>
+<contactref element="JP1" pad="3"/>
+<contactref element="IC1" pad="4"/>
+<wire x1="7.62" y1="-5.08" x2="38.1" y2="1.905" width="0" layer="19" extent="1-1"/>
+<wire x1="-1.27" y1="-14.1478" x2="7.62" y2="-5.08" width="0" layer="19" extent="1-1"/>
 </signal>
 <signal name="SHUNT-">
@@
 <contactref element="U$1" pad="P$24"/>
 </signal>
-<signal name="A0">
-<contactref element="U$1" pad="P$23"/>
-</signal>
-<signal name="A1">
-<contactref element="U$1" pad="P$22"/>
-</signal>
 <signal name="A2">
 <contactref element="U$1" pad="P$21"/>
@@
 <signal name="3.3V">
 <contactref element="U$1" pad="P$16"/>
+<contactref element="R5" pad="2"/>
+<wire x1="40.64" y1="17.145" x2="40.64" y2="12.7" width="0.8128" layer="1"/>
+<wire x1="40.64" y1="12.7" x2="38.1" y2="10.16" width="0.8128" layer="1"/>
+<wire x1="38.1" y1="10.16" x2="31.75" y2="10.16" width="0.8128" layer="1"/>
+<wire x1="30.48" y1="11.85" x2="30.48" y2="11.43" width="0.8128" layer="1"/>
+<wire x1="30.48" y1="11.43" x2="31.75" y2="10.16" width="0.8128" layer="1"/>
+<wire x1="30.16" y1="11.43" x2="30.48" y2="11.85" width="0.8128" layer="1"/>
 </signal>
 <signal name="N$11">
+<contactref element="R7" pad="1"/>
+<contactref element="R8" pad="2"/>
+<wire x1="26.7462" y1="6.2738" x2="27.6225" y2="5.3975" width="0.4064" layer="1"/>
+<wire x1="30.48" y1="5.5" x2="27.625" y2="5.4" width="0.4064" layer="1"/>
+<wire x1="27.625" y1="5.4" x2="27.6225" y2="5.3975" width="0.4064" layer="1"/>
+<wire x1="33.02" y1="5.5" x2="30.48" y2="5.5" width="0.4064" layer="1"/>
+<contactref element="IC1" pad="6"/>
+<wire x1="0" y1="-14.1478" x2="26.7462" y2="6.2738" width="0" layer="19" extent="1-1"/>
+</signal>
+<signal name="BATTERY_3.3">
+<contactref element="U$1" pad="P$23"/>
+<wire x1="15.24" y1="13.97" x2="16.51" y2="15.24" width="0.4064" layer="1"/>
+<wire x1="16.51" y1="15.24" x2="21.59" y2="15.24" width="0.4064" layer="1"/>
+<wire x1="22.86" y1="17.145" x2="22.86" y2="16.51" width="0.4064" layer="1"/>
+<wire x1="22.86" y1="16.51" x2="21.59" y2="15.24" width="0.4064" layer="1"/>
+<wire x1="21.5138" y1="12.3063" x2="21.59" y2="12.3825" width="0.4064" layer="1"/>
+<via x="21.59" y="12.3825" extent="1-16" drill="0.6"/>
+<wire x1="21.59" y1="12.3825" x2="21.59" y2="13.97" width="0.4064" layer="16"/>
+<wire x1="21.59" y1="13.97" x2="22.86" y2="15.24" width="0.4064" layer="16"/>
+<wire x1="22.86" y1="15.24" x2="22.86" y2="17.145" width="0.4064" layer="16"/>
+<contactref element="IC1" pad="1"/>
+<contactref element="R3" pad="1"/>
+<wire x1="-3.175" y1="-14.1478" x2="-4.66" y2="-27.94" width="0" layer="19" extent="1-1"/>
+<wire x1="15.24" y1="13.97" x2="-3.175" y2="-14.1478" width="0" layer="19" extent="1-1"/>
+</signal>
+<signal name="BIAS">
+<contactref element="R6" pad="2"/>
+<contactref element="R5" pad="1"/>
+<wire x1="30.48" y1="13.55" x2="33.02" y2="13.55" width="0.4064" layer="1"/>
+<contactref element="R4" pad="2"/>
+<wire x1="-2.96" y1="-33.02" x2="30.48" y2="13.55" width="0" layer="19" extent="1-1"/>
+</signal>
+<signal name="THROTTLE_IN_5">
+<contactref element="R7" pad="2"/>
+<contactref element="JP1" pad="2"/>
+<wire x1="5.08" y1="-5.08" x2="30.48" y2="7.2" width="0" layer="19" extent="1-1"/>
+</signal>
+<signal name="THROTTLE_IN_3.3">
+<contactref element="U$1" pad="P$22"/>
+<contactref element="IC1" pad="5"/>
+<contactref element="IC1" pad="7"/>
+<wire x1="0.635" y1="-14.1478" x2="25.4" y2="17.145" width="0" layer="19" extent="1-1"/>
+<wire x1="-0.635" y1="-14.1478" x2="0.635" y2="-14.1478" width="0" layer="19" extent="1-1"/>
+</signal>
+<signal name="THROTTLE_OUT_3.3">
+<contactref element="IC1" pad="10"/>
+<contactref element="IC1" pad="8"/>
+<contactref element="R9" pad="2"/>
+<wire x1="-0.635" y1="-8.7122" x2="-2.96" y2="-17.78" width="0" layer="19" extent="1-1"/>
+<wire x1="0.635" y1="-8.7122" x2="-0.635" y2="-8.7122" width="0" layer="19" extent="1-1"/>
+</signal>
+<signal name="N$1">
+<contactref element="IC1" pad="9"/>
+<contactref element="R10" pad="2"/>
+<contactref element="R9" pad="1"/>
+<wire x1="-4.66" y1="-17.78" x2="-2.96" y2="-22.86" width="0" layer="19" extent="1-1"/>
+<wire x1="0" y1="-8.7122" x2="-4.66" y2="-17.78" width="0" layer="19" extent="1-1"/>
+</signal>
+<signal name="N$2">
+<contactref element="R1" pad="2"/>
+<contactref element="R2" pad="1"/>
+<wire x1="15.24" y1="7.2" x2="17.78" y2="7.2" width="0.4064" layer="1"/>
+<wire x1="19.37" y1="8.89" x2="17.78" y2="7.2" width="0.4064" layer="1"/>
+<contactref element="IC1" pad="3"/>
+<wire x1="-1.905" y1="-14.1478" x2="15.24" y2="7.2" width="0" layer="19" extent="1-1"/>
+</signal>
+<signal name="N$3">
+<contactref element="R4" pad="1"/>
+<contactref element="IC1" pad="2"/>
+<contactref element="R3" pad="2"/>
+<wire x1="-2.96" y1="-27.94" x2="-4.66" y2="-33.02" width="0" layer="19" extent="1-1"/>
+<wire x1="-2.54" y1="-14.1478" x2="-2.96" y2="-27.94" width="0" layer="19" extent="1-1"/>
 </signal>
 </signals>

Commit message: Unsure what all has changed…
Parts:
- added C1: 100nF, rcl:C0603
- added C2: (no value), rcl:C0603
- added R11: 60K, rcl:R0603
- moved JP1 41.2 mm to (41.9, 6.99), turned to 90 degrees
- moved IC1 32.9 mm to (24.1, 9.53)
Connections:
- net 5V: now also C1.1
- net GND: now also C1.2
- net THROTTLE_OUT_3.3: no longer IC1.8, R9.2
- net THROTTLE_OUT_5: now also IC1.8, R9.2
Routing:
- net V_BATT: track 18.0 -> 0.00 mm
- net 3.3V: track 17.1 -> 0.00 mm
- net BATTERY_3.3: track 14.7 -> 0.00 mm, vias 1 -> 0
- net N$11: track 6.64 -> 0.00 mm
- net N$2: track 4.86 -> 0.00 mm
- net BIAS: track 2.54 -> 0.00 mm
Changed lines of the file:
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@@
 <element name="R7" library="rcl" package="R0603" value="1K" x="30.48" y="6.35" rot="R90"/>
 <element name="R8" library="rcl" package="R0603" value="2K" x="33.02" y="6.35" rot="R270"/>
-<element name="JP1" library="SparkFun-Connectors" package="1X03" value="" x="2.54" y="-5.08"/>
-<element name="IC1" library="linear" package="TSSOP14" value="LMV324MZ" x="-1.27" y="-11.43"/>
+<element name="JP1" library="SparkFun-Connectors" package="1X03" value="" x="41.91" y="6.985" rot="R90"/>
+<element name="IC1" library="linear" package="TSSOP14" value="LMV324MZ" x="24.13" y="9.525"/>
 <element name="R9" library="rcl" package="R0603" value="600" x="-3.81" y="-17.78"/>
 <element name="R10" library="rcl" package="R0603" value="600" x="-3.81" y="-22.86"/>
 <element name="R3" library="rcl" package="R0603" value="50K" x="-3.81" y="-27.94"/>
 <element name="R4" library="rcl" package="R0603" value="10K" x="-3.81" y="-33.02"/>
+<element name="R11" library="rcl" package="R0603" value="60K" x="-3.81" y="-38.1"/>
+<element name="C2" library="rcl" package="C0603" value="" x="-3.81" y="-43.18"/>
+<element name="C1" library="rcl" package="C0603" value="100nF" x="-3.81" y="-46.99"/>
 </elements>
 <signals>
@@
 <contactref element="IC1" pad="11"/>
 <contactref element="R10" pad="1"/>
-<wire x1="33.02" y1="11.85" x2="43.18" y2="17.145" width="0" layer="19" extent="1-1"/>
-<wire x1="33.02" y1="7.2" x2="33.02" y2="11.85" width="0" layer="19" extent="1-1"/>
-<wire x1="40.64" y1="1.905" x2="33.02" y2="7.2" width="0" layer="19" extent="1-1"/>
-<wire x1="43.18" y1="1.905" x2="40.64" y2="1.905" width="0" layer="19" extent="1-1"/>
-<wire x1="17.78" y1="5.5" x2="33.02" y2="7.2" width="0" layer="19" extent="1-1"/>
-<wire x1="3.81" y1="13.335" x2="17.78" y2="5.5" width="0" layer="19" extent="1-1"/>
-<wire x1="2.54" y1="-5.08" x2="3.81" y2="13.335" width="0" layer="19" extent="1-1"/>
-<wire x1="-1.27" y1="-8.7122" x2="2.54" y2="-5.08" width="0" layer="19" extent="1-1"/>
-<wire x1="-4.66" y1="-22.86" x2="-1.27" y2="-8.7122" width="0" layer="19" extent="1-1"/>
+<contactref element="C1" pad="2"/>
+<wire x1="-4.66" y1="-22.86" x2="-2.96" y2="-46.99" width="0" layer="19" extent="1-1"/>
+<wire x1="17.78" y1="5.5" x2="-4.66" y2="-22.86" width="0" layer="19" extent="1-1"/>
 </signal>
 <signal name="V_BATT">
 <contactref element="JP3" pad="1"/>
 <contactref element="R1" pad="1"/>
-<wire x1="3.81" y1="15.875" x2="5.715" y2="15.875" width="1.016" layer="1"/>
-<wire x1="5.715" y1="15.875" x2="7.62" y2="13.97" width="1.016" layer="1"/>
-<wire x1="7.62" y1="13.97" x2="7.62" y2="10.16" width="1.016" layer="1"/>
-<wire x1="7.62" y1="10.16" x2="12.38" y2="5.4" width="1.016" layer="1"/>
-<wire x1="15.24" y1="5.5" x2="12.38" y2="5.4" width="1.016" layer="1"/>
+<wire x1="3.81" y1="15.875" x2="15.24" y2="5.5" width="0" layer="19" extent="1-1"/>
 </signal>
 <signal name="5V">
@@
 <contactref element="JP1" pad="3"/>
 <contactref element="IC1" pad="4"/>
-<wire x1="7.62" y1="-5.08" x2="38.1" y2="1.905" width="0" layer="19" extent="1-1"/>
-<wire x1="-1.27" y1="-14.1478" x2="7.62" y2="-5.08" width="0" layer="19" extent="1-1"/>
+<contactref element="C1" pad="1"/>
+<wire x1="38.1" y1="1.905" x2="41.91" y2="12.065" width="0" layer="19" extent="1-1"/>
+<wire x1="24.13" y1="6.8072" x2="38.1" y2="1.905" width="0" layer="19" extent="1-1"/>
+<wire x1="-4.66" y1="-46.99" x2="24.13" y2="6.8072" width="0" layer="19" extent="1-1"/>
 </signal>
 <signal name="SHUNT-">
@@
 <signal name="THROTTLE_OUT_5">
 <contactref element="JP3" pad="6"/>
+<contactref element="IC1" pad="8"/>
+<contactref element="R9" pad="2"/>
+<wire x1="3.81" y1="3.175" x2="26.035" y2="12.2428" width="0" layer="19" extent="1-1"/>
+<wire x1="-2.96" y1="-17.78" x2="3.81" y2="3.175" width="0" layer="19" extent="1-1"/>
 </signal>
 <signal name="D8/A8">
@@
 <contactref element="U$1" pad="P$16"/>
 <contactref element="R5" pad="2"/>
-<wire x1="40.64" y1="17.145" x2="40.64" y2="12.7" width="0.8128" layer="1"/>
-<wire x1="40.64" y1="12.7" x2="38.1" y2="10.16" width="0.8128" layer="1"/>
-<wire x1="38.1" y1="10.16" x2="31.75" y2="10.16" width="0.8128" layer="1"/>
-<wire x1="30.48" y1="11.85" x2="30.48" y2="11.43" width="0.8128" layer="1"/>
-<wire x1="30.48" y1="11.43" x2="31.75" y2="10.16" width="0.8128" layer="1"/>
-<wire x1="30.16" y1="11.43" x2="30.48" y2="11.85" width="0.8128" layer="1"/>
+<wire x1="30.48" y1="11.85" x2="40.64" y2="17.145" width="0" layer="19" extent="1-1"/>
 </signal>
 <signal name="N$11">
 <contactref element="R7" pad="1"/>
 <contactref element="R8" pad="2"/>
-<wire x1="26.7462" y1="6.2738" x2="27.6225" y2="5.3975" width="0.4064" layer="1"/>
-<wire x1="30.48" y1="5.5" x2="27.625" y2="5.4" width="0.4064" layer="1"/>
-<wire x1="27.625" y1="5.4" x2="27.6225" y2="5.3975" width="0.4064" layer="1"/>
-<wire x1="33.02" y1="5.5" x2="30.48" y2="5.5" width="0.4064" layer="1"/>
 <contactref element="IC1" pad="6"/>
-<wire x1="0" y1="-14.1478" x2="26.7462" y2="6.2738" width="0" layer="19" extent="1-1"/>
+<wire x1="30.48" y1="5.5" x2="33.02" y2="5.5" width="0" layer="19" extent="1-1"/>
+<wire x1="25.4" y1="6.8072" x2="30.48" y2="5.5" width="0" layer="19" extent="1-1"/>
 </signal>
 <signal name="BATTERY_3.3">
 <contactref element="U$1" pad="P$23"/>
-<wire x1="15.24" y1="13.97" x2="16.51" y2="15.24" width="0.4064" layer="1"/>
-<wire x1="16.51" y1="15.24" x2="21.59" y2="15.24" width="0.4064" layer="1"/>
-<wire x1="22.86" y1="17.145" x2="22.86" y2="16.51" width="0.4064" layer="1"/>
-<wire x1="22.86" y1="16.51" x2="21.59" y2="15.24" width="0.4064" layer="1"/>
-<wire x1="21.5138" y1="12.3063" x2="21.59" y2="12.3825" width="0.4064" layer="1"/>
-<via x="21.59" y="12.3825" extent="1-16" drill="0.6"/>
-<wire x1="21.59" y1="12.3825" x2="21.59" y2="13.97" width="0.4064" layer="16"/>
-<wire x1="21.59" y1="13.97" x2="22.86" y2="15.24" width="0.4064" layer="16"/>
-<wire x1="22.86" y1="15.24" x2="22.86" y2="17.145" width="0.4064" layer="16"/>
 <contactref element="IC1" pad="1"/>
 <contactref element="R3" pad="1"/>
-<wire x1="-3.175" y1="-14.1478" x2="-4.66" y2="-27.94" width="0" layer="19" extent="1-1"/>
-<wire x1="15.24" y1="13.97" x2="-3.175" y2="-14.1478" width="0" layer="19" extent="1-1"/>
+<wire x1="22.225" y1="6.8072" x2="22.86" y2="17.145" width="0" layer="19" extent="1-1"/>
+<wire x1="-4.66" y1="-27.94" x2="22.225" y2="6.8072" width="0" layer="19" extent="1-1"/>
 </signal>
 <signal name="BIAS">
 <contactref element="R6" pad="2"/>
 <contactref element="R5" pad="1"/>
-<wire x1="30.48" y1="13.55" x2="33.02" y2="13.55" width="0.4064" layer="1"/>
 <contactref element="R4" pad="2"/>
+<wire x1="30.48" y1="13.55" x2="33.02" y2="13.55" width="0" layer="19" extent="1-1"/>
 <wire x1="-2.96" y1="-33.02" x2="30.48" y2="13.55" width="0" layer="19" extent="1-1"/>
 </signal>
@@
 <contactref element="R7" pad="2"/>
 <contactref element="JP1" pad="2"/>
-<wire x1="5.08" y1="-5.08" x2="30.48" y2="7.2" width="0" layer="19" extent="1-1"/>
+<wire x1="30.48" y1="7.2" x2="41.91" y2="9.525" width="0" layer="19" extent="1-1"/>
 </signal>
 <signal name="THROTTLE_IN_3.3">
@@
 <contactref element="IC1" pad="5"/>
 <contactref element="IC1" pad="7"/>
-<wire x1="0.635" y1="-14.1478" x2="25.4" y2="17.145" width="0" layer="19" extent="1-1"/>
-<wire x1="-0.635" y1="-14.1478" x2="0.635" y2="-14.1478" width="0" layer="19" extent="1-1"/>
+<wire x1="26.035" y1="6.8072" x2="25.4" y2="17.145" width="0" layer="19" extent="1-1"/>
+<wire x1="24.765" y1="6.8072" x2="26.035" y2="6.8072" width="0" layer="19" extent="1-1"/>
 </signal>
 <signal name="THROTTLE_OUT_3.3">
 <contactref element="IC1" pad="10"/>
-<contactref element="IC1" pad="8"/>
-<contactref element="R9" pad="2"/>
-<wire x1="-0.635" y1="-8.7122" x2="-2.96" y2="-17.78" width="0" layer="19" extent="1-1"/>
-<wire x1="0.635" y1="-8.7122" x2="-0.635" y2="-8.7122" width="0" layer="19" extent="1-1"/>
 </signal>
 <signal name="N$1">
@@
 <contactref element="R10" pad="2"/>
 <contactref element="R9" pad="1"/>
-<wire x1="-4.66" y1="-17.78" x2="-2.96" y2="-22.86" width="0" layer="19" extent="1-1"/>
-<wire x1="0" y1="-8.7122" x2="-4.66" y2="-17.78" width="0" layer="19" extent="1-1"/>
+<wire x1="-4.66" y1="-17.78" x2="25.4" y2="12.2428" width="0" layer="19" extent="1-1"/>
+<wire x1="-2.96" y1="-22.86" x2="-4.66" y2="-17.78" width="0" layer="19" extent="1-1"/>
 </signal>
 <signal name="N$2">
 <contactref element="R1" pad="2"/>
 <contactref element="R2" pad="1"/>
-<wire x1="15.24" y1="7.2" x2="17.78" y2="7.2" width="0.4064" layer="1"/>
-<wire x1="19.37" y1="8.89" x2="17.78" y2="7.2" width="0.4064" layer="1"/>
 <contactref element="IC1" pad="3"/>
-<wire x1="-1.905" y1="-14.1478" x2="15.24" y2="7.2" width="0" layer="19" extent="1-1"/>
+<wire x1="17.78" y1="7.2" x2="23.495" y2="6.8072" width="0" layer="19" extent="1-1"/>
+<wire x1="15.24" y1="7.2" x2="17.78" y2="7.2" width="0" layer="19" extent="1-1"/>
 </signal>
 <signal name="N$3">
@@
 <contactref element="R3" pad="2"/>
 <wire x1="-2.96" y1="-27.94" x2="-4.66" y2="-33.02" width="0" layer="19" extent="1-1"/>
-<wire x1="-2.54" y1="-14.1478" x2="-2.96" y2="-27.94" width="0" layer="19" extent="1-1"/>
+<wire x1="22.86" y1="6.8072" x2="-2.96" y2="-27.94" width="0" layer="19" extent="1-1"/>
 </signal>
 </signals>
