File: hardware/bicicletta-sensor.sch (EAGLE design)
At the start: 2 parts

Commit message: Better analog design. Still working on DAC for throttle output.
Parts:
- added IC1: LMV324MZ, linear:LMV324MZ
- added JP1: (no value), SparkFun-Connectors:M03PTH
- added R1: 60K, rcl:R-US_R0603
- added R10, R9: 600, rcl:R-US_R0603
- added R2: 3K, rcl:R-US_R0603
- added R3: 50K, rcl:R-US_R0603
- added R4, R5: 10K, rcl:R-US_R0603
- added R6: 5.8K, rcl:R-US_R0603
- added R7: 1K, rcl:R-US_R0603
- added R8: 2K, rcl:R-US_R0603
Connections:
- removed net A0: U$1.A0
- removed net A1: U$1.A1
- new net BATTERY_3.3: IC1A.OUT, R3.1, U$1.A0
- new net BIAS: R4.2, R5.1, R6.2
- new net N$1: IC1C.-IN, R10.2, R9.1
- new net N$11: IC1B.-IN, R7.1, R8.2
- new net N$2: IC1A.+IN, R1.2, R2.1
- new net N$3: IC1A.-IN, R3.2, R4.1
- new net THROTTLE_IN_3.3: IC1B.+IN, IC1B.OUT, U$1.A1
- new net THROTTLE_IN_5: JP1.2, R7.2
- new net THROTTLE_OUT_3.3: IC1C.+IN, IC1C.OUT, R9.2
- net 3.3V: now also R5.2
- net 5V: now also IC1P.V+, JP1.3
- net GND: now also IC1P.V-, JP1.1, R10.1, R2.2, R6.1, R8.1
- net V_BATT: now also R1.1
Other:
- note added: "IN: 38V - 58V"
- note added: "OUT: 0.5V - 2.85V"

Commit message: Unsure what all has changed…
Parts:
- added C1: 100nF, rcl:C-USC0603
- added C2: (no value), rcl:C-USC0603
- added R11: 60K, rcl:R-US_R0603
Connections:
- net 5V: now also C1.1
- net GND: now also C1.2
- net THROTTLE_OUT_3.3: no longer IC1C.OUT, R9.2
- net THROTTLE_OUT_5: now also IC1C.OUT, R9.2
Changed lines of the file:
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@@
 <part name="R3" library="rcl" deviceset="R-US_" device="R0603" value="50K"/>
 <part name="R4" library="rcl" deviceset="R-US_" device="R0603" value="10K"/>
+<part name="R11" library="rcl" deviceset="R-US_" device="R0603" value="60K"/>
+<part name="C2" library="rcl" deviceset="C-US" device="C0603"/>
+<part name="C1" library="rcl" deviceset="C-US" device="C0603" value="100nF"/>
+<part name="U$5" library="SparkFun-Aesthetics" deviceset="5V" device=""/>
+<part name="GND4" library="SparkFun-Aesthetics" deviceset="GND" device=""/>
 </parts>
 <sheets>
@@
 <instance part="R3" gate="G$1" x="96.52" y="101.6" rot="R180"/>
 <instance part="R4" gate="G$1" x="81.28" y="116.84" rot="R180"/>
+<instance part="R11" gate="G$1" x="152.4" y="149.86"/>
+<instance part="C2" gate="G$1" x="162.56" y="149.86"/>
+<instance part="C1" gate="G$1" x="129.54" y="104.14"/>
+<instance part="U$5" gate="G$1" x="129.54" y="111.76"/>
+<instance part="GND4" gate="1" x="129.54" y="93.98"/>
 </instances>
 <busses>
@@
 <pinref part="GND1" gate="1" pin="GND"/>
 </segment>
+<segment>
+<pinref part="GND4" gate="1" pin="GND"/>
+<pinref part="C1" gate="G$1" pin="2"/>
+<wire x1="129.54" y1="99.06" x2="129.54" y2="96.52" width="0.1524" layer="91"/>
+</segment>
 </net>
 <net name="~D9/A9" class="0">
@@
 <pinref part="U$3" gate="G$1" pin="5V"/>
 </segment>
+<segment>
+<pinref part="U$5" gate="G$1" pin="5V"/>
+<pinref part="C1" gate="G$1" pin="1"/>
+<wire x1="129.54" y1="106.68" x2="129.54" y2="111.76" width="0.1524" layer="91"/>
+</segment>
 </net>
 <net name="SHUNT-" class="0">
@@
 <wire x1="45.72" y1="205.74" x2="81.28" y2="205.74" width="0.1524" layer="91"/>
 <label x="55.88" y="205.74" size="1.778" layer="95"/>
+</segment>
+<segment>
+<pinref part="IC1" gate="C" pin="OUT"/>
+<wire x1="193.04" y1="134.62" x2="195.58" y2="134.62" width="0.1524" layer="91"/>
+<wire x1="195.58" y1="134.62" x2="215.9" y2="134.62" width="0.1524" layer="91"/>
+<wire x1="195.58" y1="134.62" x2="195.58" y2="121.92" width="0.1524" layer="91"/>
+<pinref part="R9" gate="G$1" pin="2"/>
+<wire x1="195.58" y1="121.92" x2="190.5" y2="121.92" width="0.1524" layer="91"/>
+<junction x="195.58" y="134.62"/>
+<label x="200.66" y="134.62" size="1.778" layer="95"/>
 </segment>
 </net>
@@
 <label x="152.4" y="137.16" size="1.778" layer="95"/>
 </segment>
-<segment>
-<pinref part="IC1" gate="C" pin="OUT"/>
-<wire x1="193.04" y1="134.62" x2="195.58" y2="134.62" width="0.1524" layer="91"/>
-<wire x1="195.58" y1="134.62" x2="215.9" y2="134.62" width="0.1524" layer="91"/>
-<wire x1="195.58" y1="134.62" x2="195.58" y2="121.92" width="0.1524" layer="91"/>
-<pinref part="R9" gate="G$1" pin="2"/>
-<wire x1="195.58" y1="121.92" x2="190.5" y2="121.92" width="0.1524" layer="91"/>
-<junction x="195.58" y="134.62"/>
-<label x="200.66" y="134.62" size="1.778" layer="95"/>
-</segment>
-</net>
+</net>
